Commit message: fixed typo

File: vsa_3dof_arm_description/urdf/qb/body_defs.urdf.xacro (robot description, xacro)
@@ -38,5 +38,5 @@
 				<origin xyz="0 0 0" rpy="0 0 0" />
 				<geometry>
-	            	<mesh filename="package://body_description/meshes/qb/cube.stl" />
+	            	<mesh filename="package://vsa_3dof_arm_description/meshes/qb/cube.stl" />
 				</geometry>
 			<material name="DLR/Blue" />

Commit message: Added individual joint limits to the qb cube URDF

File: vsa_3dof_arm_description/urdf/qb/body_defs.urdf.xacro (robot description, xacro)
@@ -2,4 +2,5 @@
 <robot xmlns:xacro="http://ros.org/wiki/xacro">
 <!-- constants -->
+	<!--FIXME: Add different joint limits for each cube -->
 	<xacro:property name="damping_all" value="1" />
 	<xacro:property name="pi" value="3.1415926535897931" />
@@ -27,6 +28,6 @@
 	<xacro:property name="length" value="64" />
 	<xacro:property name="width" value="64" />
-<!-- Definiton of the QB cube -->
-	<xacro:macro name="cube" params="parent name position orientation" >
+<!-- Definition of the QB cube -->
+	<xacro:macro name="cube" params="parent name position orientation low_limit high_limit" >
 		<joint name="${name}_dummy_joint" type="fixed" >
 			<origin xyz="${position}" rpy="${orientation}" />
@@ -55,5 +56,5 @@
 			<axis xyz="0 0 1" />
 			<dynamics damping="${damping_all}" />
-			<limit lower="${low_b * pi / 180}" upper="${up_b * pi / 180}" effort="${effort}" velocity="${velocity}"/>
+			<limit lower="${low_limit * pi / 180}" upper="${high_limit * pi / 180}" effort="${effort}" velocity="${velocity}"/>
 		</joint>
 		<link name="${name}_link">
@@ -72,11 +73,11 @@
 		<link name="${name}_dummy_link"/>
 		<xacro:cube parent="${name}_dummy_link" name="${name}_1"
-                  position="0 0 0" orientation="0 0 0" />
+                  position="0 0 0" orientation="0 0 0" low_limit="-90" high_limit="90" />
 		<xacro:cube parent="${name}_1_link" name="${name}_2"
-                  position="${c_flange/scale_f} 0 0" orientation="0 0 0" />
+                  position="${c_flange/scale_f} 0 0" orientation="0 0 0" low_limit="-115" high_limit="115" />
 		<xacro:cube parent="${name}_2_link" name="${name}_3"
-                  position="${c_flange/scale_f} 0 0" orientation="0 0 0" />
+                  position="${c_flange/scale_f} 0 0" orientation="0 0 0"  low_limit="-160" high_limit="160"/>
 		<xacro:cube parent="${name}_3_link" name="${name}_4"
-                  position="0 0 ${one_flange/scale_f} " orientation="${pi / 2} 0 0" />
+                  position="0 0 ${one_flange/scale_f} " orientation="${pi / 2} 0 0"  low_limit="-90" high_limit="90"/>
                 <link name="${name}_fixed_finger"/>
                 <joint name="${name}_fixed_finger_joint" type="fixed" >

Commit message: Fix the position of the movable finger. Range: 0->45deg

File: vsa_3dof_arm_description/urdf/qb/body_defs.urdf.xacro (robot description, xacro)
@@ -88,5 +88,5 @@
                 <link name="${name}_rotating_finger"/>
                 <joint name="${name}_rotating_finger_joint" type="fixed" >
-                    <origin xyz="0 0.1 0" rpy="${- pi/2} 0  0"/>
+                    <origin xyz="${0.1 * 0.7071} ${0.1 * 0.7071} 0" rpy="${- pi/2} 0  ${- pi/4}"/>
                     <parent link="${name}_4_link" />
                     <child link="${name}_rotating_finger" />
