Commit message: Adjust positions according to the paper

File: vsa_3dof_arm_description/urdf/qb/body.urdf.xacro (robot description, xacro)
@@ -5,4 +5,5 @@
   <xacro:property name="cube_size" value="66" />
   <xacro:property name="arm_height" value="0.3" />
+  <xacro:property name="holder_height" value="0.089" />
   <xacro:include filename="$(find vsa_3dof_arm_description)/urdf/qb/body_defs.urdf.xacro"/>
   <xacro:include filename="$(find vsa_3dof_arm_description)/urdf/materials.urdf.xacro"/>
@@ -51,5 +52,5 @@
       <origin xyz="0 0 0" rpy="0 0 0"/>
       <geometry>
-        <sphere radius="0.03"/>
+        <sphere radius="0.01"/>
       </geometry>
       <material name="Green">
@@ -60,10 +61,10 @@
       	    <origin xyz="0 0 0" rpy="0 0 0"/>
             <geometry>
-              <sphere radius="0.03"/>
+              <sphere radius="0.01"/>
             </geometry>
     	</collision>
   </link>
   <joint name="left_holder_joint" type="fixed" >
-      <origin xyz="0 -0.15 0.089" rpy="0 0 0"/>
+      <origin xyz="${0.044 + 0.030} -0.16 ${holder_height}" rpy="0 0 0"/>
       <parent link="base_link" />
       <child link="left_holder_link" />
@@ -74,5 +75,5 @@
       <origin xyz="0 0 0" rpy="0 0 0"/>
       <geometry>
-        <sphere radius="0.03"/>
+        <sphere radius="0.01"/>
       </geometry>
       <material name="Red">
@@ -83,10 +84,10 @@
       	    <origin xyz="0 0 0" rpy="0 0 0"/>
             <geometry>
-              <sphere radius="0.03"/>
+              <sphere radius="0.01"/>
             </geometry>
     	</collision>
   </link>
   <joint name="right_holder_joint" type="fixed" >
-      <origin xyz="0 0.15 0.089" rpy="0 0 0"/>
+      <origin xyz="${0.044 + 0.030} 0.16 ${holder_height}" rpy="0 0 0"/>
       <parent link="base_link" />
       <child link="right_holder_link" />
@@ -95,8 +96,15 @@
   <link name="arm_mounting_frame"/>
   <joint name="arm_mounting_joint" type="fixed" >
-      <origin xyz="0.088 0 ${- cube_size/2/scale_f + arm_height}" rpy="${pi} 0 0"/>
+      <origin xyz="${0.044 + 0.0535 - cube_size/2/scale_f} 0 ${- cube_size/2/scale_f + arm_height}" rpy="${pi} 0 0"/>
       <parent link="base_link" />
       <child link="arm_mounting_frame" />
   </joint>
-  <xacro:vsa_3dof_arm parent="arm_mounting_frame" name="3dof_arm"/>
+  <xacro:vsa_3dof_arm parent="arm_mounting_frame" name="arm"/>
+  <!-- Adding a link at the only height the arm can reach -->
+  <link name="base_link_zero"/>
+  <joint name="base_link_zero_joint" type="fixed">
+    <origin xyz="0 0 ${-holder_height}" rpy="0 0 0"/>
+      <parent link="base_link_zero" />
+      <child link="base_link" />
+  </joint>
 </robot>

Commit message: Align the holder_link frames to easily reachable orientations

File: vsa_3dof_arm_description/urdf/qb/body.urdf.xacro (robot description, xacro)
@@ -66,5 +66,5 @@
   </link>
   <joint name="left_holder_joint" type="fixed" >
-      <origin xyz="${0.044 + 0.030} -0.16 ${holder_height}" rpy="0 0 0"/>
+      <origin xyz="${0.044 + 0.030} -0.16 ${holder_height}" rpy="${pi} 0 ${-pi/2}"/>
       <parent link="base_link" />
       <child link="left_holder_link" />
@@ -89,5 +89,5 @@
   </link>
   <joint name="right_holder_joint" type="fixed" >
-      <origin xyz="${0.044 + 0.030} 0.16 ${holder_height}" rpy="0 0 0"/>
+      <origin xyz="${0.044 + 0.030} 0.16 ${holder_height}" rpy="${pi} 0 ${pi/2}"/>
       <parent link="base_link" />
       <child link="right_holder_link" />

Commit message: Corrected size of the metal bars in URDF

File: vsa_3dof_arm_description/urdf/qb/body.urdf.xacro (robot description, xacro)
@@ -10,7 +10,7 @@
   <link name="base_link">
     <visual>
-      <origin xyz="0 0 0.25" rpy="0 0 0"/>
+      <origin xyz="0 0 0.2" rpy="0 0 0"/>
       <geometry>
-        <box size="0.088 0.088 0.5"/>
+        <box size="0.060 0.060 0.4"/>
       </geometry>
       <material name="Gray">
@@ -19,7 +19,7 @@
     </visual>
 	<collision>
-      		<origin xyz="0 0 0.25" rpy="0 0 0"/>
+      		<origin xyz="0 0 0.2" rpy="0 0 0"/>
       		<geometry>
-        	<box size="0.088 0.088 0.5"/>
+        	<box size="0.06 0.06 0.4"/>
      		 </geometry>
     	</collision>
@@ -27,7 +27,7 @@
   <link name="horizontal_bar_link">
     <visual>
-      <origin xyz="0 0 0.022" rpy="0 0 0"/>
+      <origin xyz="0 0 0.015" rpy="0 0 0"/>
       <geometry>
-        <box size="0.088 0.5 0.044"/>
+        <box size="0.06 0.5 0.03"/>
       </geometry>
       <material name="Gray">
@@ -36,7 +36,7 @@
     </visual>
 	<collision>
-      		<origin xyz="0 0 0.022" rpy="0 0 0"/>
+      		<origin xyz="0 0 0.015" rpy="0 0 0"/>
       		<geometry>
-        	<box size="0.088 0.5 0.044"/>
+        	<box size="0.06 0.5 0.03"/>
      		 </geometry>
     	</collision>
@@ -66,5 +66,5 @@
   </link>
   <joint name="left_holder_joint" type="fixed" >
-      <origin xyz="${0.044 + 0.030} -0.16 ${holder_height}" rpy="${pi} 0 ${-pi/2}"/>
+      <origin xyz="${0.03 + 0.030} -0.16 ${holder_height}" rpy="${pi} 0 ${-pi/2}"/>
       <parent link="base_link" />
       <child link="left_holder_link" />
@@ -89,5 +89,5 @@
   </link>
   <joint name="right_holder_joint" type="fixed" >
-      <origin xyz="${0.044 + 0.030} 0.16 ${holder_height}" rpy="${pi} 0 ${pi/2}"/>
+      <origin xyz="${0.03 + 0.030} 0.16 ${holder_height}" rpy="${pi} 0 ${pi/2}"/>
       <parent link="base_link" />
       <child link="right_holder_link" />

Commit message: Fix small offset to the holders

File: vsa_3dof_arm_description/urdf/qb/body.urdf.xacro (robot description, xacro)
@@ -66,5 +66,5 @@
   </link>
   <joint name="left_holder_joint" type="fixed" >
-      <origin xyz="${0.03 + 0.030} -0.16 ${holder_height}" rpy="${pi} 0 ${-pi/2}"/>
+      <origin xyz="${0.0345} -0.16 ${holder_height}" rpy="${pi} 0 ${-pi/2}"/>
       <parent link="base_link" />
       <child link="left_holder_link" />
@@ -89,5 +89,5 @@
   </link>
   <joint name="right_holder_joint" type="fixed" >
-      <origin xyz="${0.03 + 0.030} 0.16 ${holder_height}" rpy="${pi} 0 ${pi/2}"/>
+      <origin xyz="${0.0345} 0.16 ${holder_height}" rpy="${pi} 0 ${pi/2}"/>
       <parent link="base_link" />
       <child link="right_holder_link" />

Commit message: Fixed the offset of the holder again

File: vsa_3dof_arm_description/urdf/qb/body.urdf.xacro (robot description, xacro)
@@ -66,5 +66,5 @@
   </link>
   <joint name="left_holder_joint" type="fixed" >
-      <origin xyz="${0.0345} -0.16 ${holder_height}" rpy="${pi} 0 ${-pi/2}"/>
+      <origin xyz="${0.0415} -0.16 ${holder_height}" rpy="${pi} 0 ${-pi/2}"/>
       <parent link="base_link" />
       <child link="left_holder_link" />
@@ -89,5 +89,5 @@
   </link>
   <joint name="right_holder_joint" type="fixed" >
-      <origin xyz="${0.0345} 0.16 ${holder_height}" rpy="${pi} 0 ${pi/2}"/>
+      <origin xyz="${0.0415} 0.16 ${holder_height}" rpy="${pi} 0 ${pi/2}"/>
       <parent link="base_link" />
       <child link="right_holder_link" />
